File: A_Micromouse_Team_PCB_Rev1/A_Micromouse_Team_PCB_Rev1.kicad_pcb (KiCad board)
At the start: 2 copper layers, 13 parts, among them J1 Conn_01x07_Pin, J10 Conn_01x06, J2 Conn_01x07_Pin, J3 Conn_01x07_Pin, J4 Conn_01x07_Pin, J5 Conn_01x06_Pin, J6 Conn_01x06_Pin, J7 Conn_01x04_Socket, J8 Conn_01x07_Pin, J9 Conn_01x02_Socket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

Commit message: changed Net Classes
Parts:
- moved J8 24.0 mm to (132.1, 73.7), turned to 180 degrees
Routing:
- net +5V: track 0.00 -> 79.7 mm, vias 0 -> 3
- net Net-(J5-Pin_5): track 0.00 -> 20.7 mm, vias 0 -> 1
- net Net-(J5-Pin_3): track 0.00 -> 19.3 mm
- net GND: track 0.00 -> 5.56 mm
Changed lines of the file:
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@@
   )
   (footprint "Connector_PinHeader_2.54mm:PinHeader_1x07_P2.54mm_Vertical" (layer "F.Cu")
-    (at 119.38 53.34)
+    (at 132.08 73.66 180)
     (descr "Through hole straight pin header, 1x07, 2.54mm pitch, single row")
     (tags "Through hole pin header THT 1x07 2.54mm single row")
@@
     (fp_line (start 1.27 16.51) (end -1.27 16.51)
       (stroke (width 0.1) (type solid)) (layer "F.Fab"))
-    (pad "1" thru_hole rect (at 0 0) (size 1.7 1.7) (drill 1) (layers "*.Cu" "*.Mask")
+    (pad "1" thru_hole rect (at 0 0 180) (size 1.7 1.7) (drill 1) (layers "*.Cu" "*.Mask")
       (net 23 "unconnected-(J8-Pin_1-Pad1)") (pinfunction "Pin_1") (pintype "passive+no_connect"))
-    (pad "2" thru_hole oval (at 0 2.54) (size 1.7 1.7) (drill 1) (layers "*.Cu" "*.Mask")
+    (pad "2" thru_hole oval (at 0 2.54 180) (size 1.7 1.7) (drill 1) (layers "*.Cu" "*.Mask")
       (net 2 "+5V") (pinfunction "Pin_2") (pintype "passive"))
-    (pad "3" thru_hole oval (at 0 5.08) (size 1.7 1.7) (drill 1) (layers "*.Cu" "*.Mask")
+    (pad "3" thru_hole oval (at 0 5.08 180) (size 1.7 1.7) (drill 1) (layers "*.Cu" "*.Mask")
       (net 3 "GND1") (pinfunction "Pin_3") (pintype "passive"))
-    (pad "4" thru_hole oval (at 0 7.62) (size 1.7 1.7) (drill 1) (layers "*.Cu" "*.Mask")
+    (pad "4" thru_hole oval (at 0 7.62 180) (size 1.7 1.7) (drill 1) (layers "*.Cu" "*.Mask")
       (net 4 "SDA") (pinfunction "Pin_4") (pintype "passive"))
-    (pad "5" thru_hole oval (at 0 10.16) (size 1.7 1.7) (drill 1) (layers "*.Cu" "*.Mask")
+    (pad "5" thru_hole oval (at 0 10.16 180) (size 1.7 1.7) (drill 1) (layers "*.Cu" "*.Mask")
       (net 5 "SCL") (pinfunction "Pin_5") (pintype "passive"))
-    (pad "6" thru_hole oval (at 0 12.7) (size 1.7 1.7) (drill 1) (layers "*.Cu" "*.Mask")
+    (pad "6" thru_hole oval (at 0 12.7 180) (size 1.7 1.7) (drill 1) (layers "*.Cu" "*.Mask")
       (net 24 "Net-(J8-Pin_6)") (pinfunction "Pin_6") (pintype "passive"))
-    (pad "7" thru_hole oval (at 0 15.24) (size 1.7 1.7) (drill 1) (layers "*.Cu" "*.Mask")
+    (pad "7" thru_hole oval (at 0 15.24 180) (size 1.7 1.7) (drill 1) (layers "*.Cu" "*.Mask")
       (net 25 "unconnected-(J8-Pin_7-Pad7)") (pinfunction "Pin_7") (pintype "passive+no_connect"))
     (model "${KICAD6_3DMODEL_DIR}/Connector_PinHeader_2.54mm.3dshapes/PinHeader_1x07_P2.54mm_Vertical.wrl"
@@
     )
   )
+  (segment (start 76.68 68.58) (end 66.04 68.58) (width 1) (layer "F.Cu") (net 2))
+  (segment (start 63.5 83.82) (end 73.66 83.82) (width 1) (layer "F.Cu") (net 2))
+  (segment (start 63.5 68.58) (end 60.96 71.12) (width 1) (layer "F.Cu") (net 2))
+  (segment (start 75.952118 69.307882) (end 75.952118 69.374656) (width 1) (layer "F.Cu") (net 2))
+  (segment (start 64.525 70.095) (end 63.5 71.12) (width 1) (layer "F.Cu") (net 2))
+  (segment (start 75.231774 70.095) (end 64.525 70.095) (width 1) (layer "F.Cu") (net 2))
+  (segment (start 75.952118 69.374656) (end 75.231774 70.095) (width 1) (layer "F.Cu") (net 2))
+  (segment (start 65.12 57.5) (end 62.47 57.5) (width 1) (layer "F.Cu") (net 2))
+  (segment (start 66.04 68.58) (end 66.04 58.42) (width 1) (layer "F.Cu") (net 2))
+  (segment (start 66.04 58.42) (end 65.12 57.5) (width 1) (layer "F.Cu") (net 2))
+  (segment (start 76.68 68.58) (end 75.952118 69.307882) (width 1) (layer "F.Cu") (net 2))
+  (segment (start 76.68 68.58) (end 63.5 68.58) (width 1) (layer "F.Cu") (net 2))
+  (via (at 63.5 71.12) (size 1.5) (drill 0.7) (layers "F.Cu" "B.Cu") (net 2))
+  (via (at 60.96 71.12) (size 1.5) (drill 0.7) (layers "F.Cu" "B.Cu") (net 2))
+  (via (at 63.5 83.82) (size 1.5) (drill 0.7) (layers "F.Cu" "B.Cu") (net 2))
+  (segment (start 60.96 81.28) (end 63.5 83.82) (width 1) (layer "B.Cu") (net 2))
+  (segment (start 60.96 71.12) (end 60.96 81.28) (width 1) (layer "B.Cu") (net 2))
+  (segment (start 76.68 60.96) (end 71.12 60.96) (width 1) (layer "F.Cu") (net 14))
+  (segment (start 68.58 58.42) (end 66.04 55.88) (width 0.25) (layer "F.Cu") (net 16))
+  (segment (start 68.58 66.04) (end 68.58 58.42) (width 0.25) (layer "F.Cu") (net 16))
+  (segment (start 76.68 66.04) (end 68.58 66.04) (width 0.25) (layer "F.Cu") (net 16))
+  (segment (start 71.12 71.12) (end 68.58 73.66) (width 0.25) (layer "F.Cu") (net 17))
+  (segment (start 76.68 71.12) (end 74.14 73.66) (width 0.25) (layer "F.Cu") (net 17))
+  (segment (start 76.68 71.12) (end 75.609973 72.190027) (width 0.25) (layer "F.Cu") (net 17))
+  (segment (start 74.14 73.66) (end 73.66 73.66) (width 0.25) (layer "F.Cu") (net 17))
+  (segment (start 76.68 71.12) (end 71.12 71.12) (width 0.25) (layer "F.Cu") (net 17))
+  (segment (start 75.609973 73.069973) (end 75.609973 72.190027) (width 0.25) (layer "F.Cu") (net 17))
+  (via (at 68.58 73.66) (size 0.8) (drill 0.4) (layers "F.Cu" "B.Cu") (net 17))
+  (segment (start 68.58 73.66) (end 68.58 78.74) (width 0.25) (layer "B.Cu") (net 17))
 )
